File: BSPD/BSPD_V2/BSPD.sch (KiCad schematic (older format))
At the start: 67 parts, among them J1 Conn_01x06_Female, J2 Conn_01x02_Female, Q1 Q_PMOS_DGS, U1 LM311, U2 LM311, U3 LM311, U4 74AUC2G08, U5 LM393, U6 LM393, U7 LM393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

Commit message: BSPD and loom documentation
Parts:
- removed D3: D_Zener_Small, Package_TO_SOT_SMD:SOT-23, symbol Device:D_Zener_Small
- removed J1: Conn_01x06_Female, Connector_Molex:Molex_Micro-Fit_3.0_43045-0600_2x03_P3.00mm_Horizontal, symbol Connector:Conn_01x06_Female
- added D3: BSPD_OK, LED_SMD:LED_0805_2012Metric, symbol Device:LED
- added D6: ~OCSC, LED_SMD:LED_0805_2012Metric, symbol Device:LED
- added D7: CURRENT THRESHOLD, LED_SMD:LED_0805_2012Metric, symbol Device:LED
- added D8: BRAKE THRESHOLD, LED_SMD:LED_0805_2012Metric, symbol Device:LED
- added J1: Conn_01x10_Female, Connector_Molex:Molex_Micro-Fit_3.0_43045-1012_2x05_P3.00mm_Vertical, symbol Connector:Conn_01x10_Female
- added R23, R24: 10K, Resistor_SMD:R_1206_3216Metric, symbol Device:R
- added R25, R26, R27, R28: R, Resistor_SMD:R_1206_3216Metric, symbol Device:R
- added U10: MCP6004, Package_SO:SOIC-14_3.9x8.7mm_P1.27mm, symbol Amplifier_Operational:MCP6004
- C3: value CP1_Small -> 0.1uF
- J2: footprint Connector_Molex:Molex_Micro-Fit_3.0_43045-0200_2x01_P3.00mm_Horizontal -> Connector_Molex:Molex_Micro-Fit_3.0_43045-0212_2x01_P3.00mm_Vertical
- R1, R10, R11, R12, R13, R14, R15, R16, R17, R18, R19, R2, R20, R21, R22, R4, R5, R7, R8, R9: footprint Resistor_SMD:R_1206_3216Metric_Pad1.42x1.75mm_HandSolder -> Resistor_SMD:R_1206_3216Metric
- R3, R6: value R -> 10K; footprint Resistor_SMD:R_1206_3216Metric_Pad1.42x1.75mm_HandSolder -> Resistor_SMD:R_1206_3216Metric
Connections:
- net BRK_FRNT: now also C1.1, C4.2, D1.1 (K), R1.1, R4.1, TP3.1, U1.3 (-), U6.3 (+), U6.6 (_)
- net BRK_REAR: now also C2.1, C5.2, D2.1 (K), R2.1, R5.1, TP4.1, U2.3 (-), U7.3 (+), U7.6 (_)
- net BRK_SIG: now also U10.12 (+)
- net BSPD_OK: now also J1.1 (Pin_1), U10.3 (+)
- net Brk_Frnt_Inp: now also R1.2, J1.6 (Pin_6); no longer C1.1, C4.2, D1.1 (K), R1.1, R4.1, TP3.1, U1.3 (-), U6.3 (+), U6.6 (_)
- net Brk_Rear_Inp: now also R2.2, J1.5 (Pin_5); no longer C2.1, C5.2, D2.1 (K), R2.1, R5.1, TP4.1, U2.3 (-), U7.3 (+), U7.6 (_)
- net CRNT_SIG: now also U10.10 (+)
- net GND: now also J1.7 (Pin_7), J1.8 (Pin_8), R23.2, R25.2, R26.2, R27.2, R28.2, U10.11 (V-); no longer R6.2, U9.6 (-)
- net VCC: now also C3.1, J1.10 (Pin_10), J1.9 (Pin_9), U10.4 (V+); no longer U9.5 (+)
- net ~OCSC: now also U10.5 (+)
- net CURRENT: now reaches U9.7
- net CURRENT: now also C8.2, TP6.1, U3.3 (-), U5.3 (+), U5.6 (_), R24.1
- net CURRENT_SIG: now reaches R3.2
- net CURRENT_SIG: now also J1.4 (Pin_4)
- removed net Crnt_Sig_Inp: C3.1, C8.2, R3.1, R6.1, TP6.1, U3.3 (-), U5.3 (+), U5.6 (_)
- new net: R24.2, R3.1, U9.5 (+)
- new net: R23.1, R6.1, U9.6 (-)
- new net: D3.2 (A), U10.1, U10.2 (-)
- new net: D6.2 (A), U10.6 (-), U10.7
- new net: D7.2 (A), U10.8, U10.9 (-)
- new net: D8.2 (A), U10.13 (-), U10.14
- new net: D3.1 (K), R25.1
- new net: D6.1 (K), R26.1
- new net: D7.1 (K), R27.1
- new net: D8.1 (K), R28.1
- new net CURRENT_REF: J1.3 (Pin_3), R6.2
Other:
- moved on the sheet: C1, C10, C11, C12, C13, C14, C15, C16, C2, C4, C5, C6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

Commit message: BSPD acc board
Parts:
- removed D4: D_Zener, Package_TO_SOT_SMD:SOT-23, symbol Device:D_Zener
- removed R23, R24: 10K, Resistor_SMD:R_1206_3216Metric, symbol Device:R
- removed R7: R, Resistor_SMD:R_1206_3216Metric, symbol Device:R
- added C17: 0.1uF, Capacitor_SMD:C_0805_2012Metric_Pad1.15x1.40mm_HandSolder, symbol BSPD-rescue:CP1_Small-Device
- added U11: AD8236ARMZ, Package_SO:SOIC-8_3.9x4.9mm_P1.27mm, symbol Amplifier_Instrumentation:AD8236ARMZ
- added U? (x4): LM393, Package_SO:SOIC-8_3.9x4.9mm_P1.27mm, symbol Comparator:LM393
- R3: value 10K -> Rg
- R6: value 10K -> 10k
- RV1, RV2, RV3: footprint Potentiometer_THT:Potentiometer_Bourns_3266Y_Vertical -> Potentiometer_THT:Potentiometer_Bourns_3296Y_Vertical
Connections:
- net BSPD_OK: now also J1.2 (Pin_2)
- net CURRENT: now also R6.1, U11.7; no longer U9.7
- net CURRENT_REF: now also U11.1 (-), U?.3 (+), U?.6 (_); no longer R6.2
- net CURRENT_SIG: now also U11.4 (+), U?.3 (+), U?.6 (_); no longer R3.2
- net GND: now also Q1.2 (G), R6.2, U9.6 (-), C17.2, U11.5 (Vs-), U11.6 (Ref)
- net OC: now also U?.2 (-), U?.2 (-)
- net SC: now also U?.5 (+), U?.5 (+)
- net VCC: now also U9.5 (+), C17.1, U11.8 (Vs+)
- net ~OCSC: now also U?.1, U?.1, U?.7, U?.7
- net at R3.1: now also U11.2 (Rg); no longer U9.5 (+)
- new net: R3.2, U11.3 (Rg)
Other:
- moved on the sheet: C1, C2, D1, D2, Q1, R1, R2, R4, R5, U9B
